File: schematics/MC68000/cpu.kicad_sch (KiCad schematic)
At the start: 52 parts, among them J2 Conn_02x37_Row_Letter_Last, SW1 Reset, U1 74LS00, U10 74LS244, U11 74LS244, U12 74LS148, U2 74LS05, U3 74LS161, U4 ICM7555xB, U5 68000D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

Commit message: Update...
Parts:
- added D1: /RESET, symbol Device:LED
- added D2: /HALT, symbol Device:LED
- added D3: ON, symbol Device:LED
- added R18, R19, R20: 470R, symbol Device:R
- renumbered C6_U1E to C6_U1E1, C7_U1E to C7_U1E1
Connections:
- net VCC is gone; now on net +5V: J2.18a (Pin_18a), J2.18b (Pin_18b)
- net /bE is gone; now on net bE: U6.12 (O3a)
- net +5V: now also D1.1 (K), D2.1 (K), D3.1 (K)
- net FC0: no longer J2.20b (Pin_20b)
- net FC1: no longer J2.21b (Pin_21b)
- net FC2: no longer J2.22b (Pin_22b)
- net GND: now also R20.2
- net R/W: no longer J2.24b (Pin_24b)
- net bFC0: now also J2.20b (Pin_20b)
- net bFC1: now also J2.21b (Pin_21b)
- net bFC2: now also J2.22b (Pin_22b)
- net bR/W: now also J2.24b (Pin_24b)
- net /HALT: now also U2.9
- net /LDS: no longer J2.15b (Pin_15b)
- net /RESET: now also R18.2
- net /UDS: no longer J2.14b (Pin_14b)
- net /VMA: no longer J2.16b (Pin_16b)
- net /bLDS: now also J2.15b (Pin_15b)
- net /bUDS: now also J2.14b (Pin_14b)
- net /bVMA: now also J2.16b (Pin_16b)
- net at U2.8: now also R19.2
- net E renamed bE
- new net: D1.2 (A), R18.1
- new net: D2.2 (A), R19.1
- new net: D3.2 (A), R20.1
Other:
- moved on the sheet: U2D
