File: schematics/MC68000/cpuNoBuffer.kicad_sch (KiCad schematic)
At the start: 45 parts, among them J10 Conn_02x37_Row_Letter_Last, SW2 Reset, U2.1 68000D, U2.2 74LS161, U2.2_C1 100nF, U2.3 74LS148, U2.3_C1 100nF, U2.4 ICM7555xB, U2.4_C1 100nF, U2.5 74LS05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

Commit message: Cpu's board tested
Connections:
- net CLK: now also U2.1.15 (CLK), X3.8 (OUT)
Other:
- note added: "0 - por o soquete do ci intrq 1 - por todos os capacitores 100nf 2 - por todos os terras 3 - por todos os vccs 4 - por todos os pullups com opção de pulldown 5 - por o oscilador 6 - por o ci intrq 7 - ligar o clock 8 - ligar a cpu ao halt reset 9 - ligar os leds"
- note added: "PARA FINS DE TESTE NO LUGAR DE /ROM_CE E /RAM_CS ESTOU USANDO O SINAL DA CPU /AS"
Changed lines of the file:
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@@
     (stroke (width 0) (type default))
+  )
+  (text "PARA FINS DE TESTE\nNO LUGAR DE /ROM_CE\nE /RAM_CS ESTOU \nUSANDO O SINAL \nDA CPU /AS \n"
+    (at 15.24 74.93 0)
+    (effects (font (size 1.27 1.27)) (justify left bottom))
   )
   (text "CPU MC68000\nINTERRUPT \nCLOCK 16MHZ\nRESET AND HALT\nDTACK GLUE LOGIC\n"
@@
     (effects (font (size 1.27 1.27) (thickness 0.254) bold) (justify left bottom))
   )
+  (text "0 - por o soquete do ci intrq\n1 - por todos os capacitores 100nf\n2 - por todos os terras\n3 - por todos os vccs\n4 - por todos os pullups com opção de pulldown\n5 - por o oscilador\n6 - por o ci intrq\n7 - ligar o clock\n8 - ligar a cpu ao halt reset\n9 - ligar os leds"
+    (at 17.78 35.56 0)
+    (effects (font (size 1.27 1.27)) (justify left bottom))
+  )
   (label "D11" (at 252.73 134.62 0) (fields_autoplaced)
     (effects (font (size 1.27 1.27)) (justify left bottom))
@@
     (effects (font (size 1.27 1.27)) (justify left bottom))
   )
+  (label "CLK" (at 153.67 45.72 0) (fields_autoplaced)
+    (effects (font (size 1.27 1.27)) (justify left bottom))
+  )

Commit message: Ram memory test 2 OK
Parts:
- added U28: 74LS05, Package_DIP:CERDIP-14_W7.62mm_SideBrazed_LongPads, symbol 74xx:74LS05
Connections:
- net /MEM_OE is gone; now on net C./DTACK: J10.35b (Pin_35b)
- net C./DTACK: no longer J10.28b (Pin_28b)
- net /RAM_CS: no longer J10.36b (Pin_36b)
- net /RESET: now also J10.37b (Pin_37b)
- net /ROM_CE: no longer J10.37b (Pin_37b)
- net /RD: now reaches J10.33b (Pin_33b)
- net /RD: now also U28.10
- net /IO_CS: now reaches J10.34b (Pin_34b)
- net /DTACK: no longer names the net of U2.2.11 (Q3)
- new net RESET: J10.36b (Pin_36b)
- new net bR/W: U28.11
