File: schematics/MC68000/cpuNoBuffer.kicad_sch (KiCad schematic)
At the start: 47 parts, among them J10 Conn_02x37_Row_Letter_Last, SW2 Reset, U2.1 68000D, U2.2 74LS161, U2.2_C1 100nF, U2.3 74LS148, U2.3_C1 100nF, U2.4 ICM7555xB, U2.4_C1 100nF, U2.5 74LS05, U2.5_C1 100nF, U2.6 74LS00, U2.6_C1 100nF, U21_C1 100nF, X3 16Mhz

Commit message: Compilando com linker
Other:
- note added: "nao estou usando o chip que pode provocar wait states nesse momento DTACK está sendo tratado na GAL"
Changed lines of the file:
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@@
     (effects (font (size 1.27 1.27) (thickness 0.254) bold) (justify left bottom))
+  )
+  (text "nao estou usando o chip que \npode provocar wait states\nnesse momento DTACK está \nsendo tratado na GAL"
+    (at 39.37 93.98 0)
+    (effects (font (size 1.27 1.27)) (justify left bottom))
   )
   (text "0 - por o soquete do ci intrq\n1 - por todos os capacitores 100nf\n2 - por todos os terras\n3 - por todos os vccs\n4 - por todos os pullups com opção de pulldown\n5 - por o oscilador\n6 - por o ci intrq\n7 - ligar o clock\n8 - ligar a cpu ao halt reset\n9 - ligar os leds"

Commit message: Updating...
Parts:
- added R51, R52: 10k, Resistor_THT:R_Axial_DIN0204_L3.6mm_D1.6mm_P5.08mm_Horizontal, symbol Device:R
- added SW3: Xmodem, Button_Switch_THT:SW_Push_1P2T_Vertical_E-Switch_800UDP8P1A1M6, symbol Switch:SW_Push
Connections:
- net +5V: now also R52.1, SW3.2
- net GND: now also R51.2
- net key_cs: now reaches J10.32b (Pin_32b)
- net key_cs: now also U2.6.10, U2.6.9
- net at U2.6.8: now also U2.6.4
- net at U2.5.5: now also U2.6.6
- net SWITCH_OUT: now reaches U2.5.6
- net SWITCH_OUT: now also R52.2
- net at U2.6.5: now also R51.1, SW3.1
Other:
- note added: "AND NAND 0 0 = 0 0 0 = 1 0 1 = 0 0 1 = 1 1 0 = 0 1 0 = 1 1 1 = 1 1 1 = 0"
- note added: "key_cs: 0 FORÇA 1 NA SAIDA"
- moved on the sheet: U2.5C, U2.6B, U2.6C

Commit message: Interrupts working...
Parts:
- removed U2.3: 74LS148, Package_DIP:CERDIP-16_W7.62mm_SideBrazed_LongPads, symbol 74xx:74LS148
- removed X3: 16Mhz, Oscillator:Oscillator_DIP-14, symbol Oscillator:ACO-xxxMHz
- added BT1: Battery, symbol Device:Battery
- added D7, D8: 1N4148, Diode_THT:D_DO-35_SOD27_P7.62mm_Horizontal, symbol Diode:1N4148
- added D9: 3V, symbol Device:D_Zener
- added Q1: NPN, symbol Simulation_SPICE:NPN
- added Q2: PNP, symbol Simulation_SPICE:PNP
- added R53, R54, R56: 10k, Resistor_THT:R_Axial_DIN0204_L3.6mm_D1.6mm_P5.08mm_Horizontal, symbol Device:R
- added R55: 100k, Resistor_THT:R_Axial_DIN0204_L3.6mm_D1.6mm_P5.08mm_Horizontal, symbol Device:R
- added R57: 1k, Resistor_THT:R_Axial_DIN0204_L3.6mm_D1.6mm_P5.08mm_Horizontal, symbol Device:R
- added R58: 4k7, Resistor_THT:R_Axial_DIN0204_L3.6mm_D1.6mm_P5.08mm_Horizontal, symbol Device:R
- added U2.7, U30, U31: 74LS138, symbol 74xx:74LS138
- added U2.7_C1, U2.8_C1, U2.9_C1, U3.0_C1: 100nF, Capacitor_SMD:C_0603_1608Metric, symbol Device:C
- added U2.8: PAL20L8, symbol Logic_Programmable:PAL20L8
- added U2.9: 8253, Package_DIP:DIP-24_W15.24mm, symbol Timer:8253
- added U26: ~, symbol OSLIB:MM58167
- added U32: 74LS148, symbol 74xx:74LS148
- added X1: 16MHZ, Oscillator:Oscillator_SMD_Abracon_ASCO-4Pin_1.6x1.2mm, symbol Oscillator:ASCO
- added X2: 32KHZ, Oscillator:Oscillator_DIP-14, symbol Oscillator:ACO-xxxMHz-A
Connections:
- net /HALT is gone; now on net /RESET: R32.2, U2.1.17 (HALT), U2.5.4, U2.5.9
- net +5V: now also U2.2.7 (CEP), U2.2.9 (~{PE}), D8.2 (A), Q2.3 (E), R53.1, R57.1, U2.7.16 (VCC), U2.7.6 (E3), U32.1 (I4), U32.16 (VCC), U32.2 (I5), U32.4 (I7), X1.4 (VDD), X2.14 (Vcc)
- net A1: now also U2.8.3 (I3), U2.9.19 (A0), U26.5 (A0), U30.1 (A0)
- net A10: now also U2.7.3 (A2)
- net A11: now also U2.7.5 (E2)
- net A2: now also U2.8.2 (I2), U2.9.20 (A1), U26.6 (A1), U30.2 (A1)
- net A3: now also U2.8.1 (I1), U26.7 (A2), U30.3 (A2)
- net A4: now also U26.8 (A3)
- net A5: now also U26.9 (A4)
- net A8: now also U2.7.1 (A0)
- net A9: now also U2.7.2 (A1)
- net C.FC0: now also U2.8.4 (I4), U31.1 (A0)
- net C.FC1: now also U2.8.5 (I5), U31.2 (A1)
- net C.FC2: now also U2.8.6 (I6), U31.3 (A2)
- net C.R/W: now also U2.9.23 (~{WR}), U26.3 (/WR)
- net C./VPA: now also U2.8.15 (IO15)
- net CLK: now also X1.3 (OUT)
- net D1: now also U2.9.8 (D0), U26.15 (D0)
- net D2: now also U2.9.7 (D1), U26.16 (D1)
- net D3: now also U2.9.6 (D2), U26.17 (D2)
- net D4: now also U2.9.5 (D3), U26.18 (D3)
- net D5: now also U2.9.4 (D4), U26.19 (D4)
- net D6: now also U2.9.3 (D5), U26.20 (D5)
- net D7: now also U2.9.2 (D6), U26.21 (D6)
- net D8: now also U2.9.1 (D7), U26.22 (D7)
- net GND: now also BT1.2 (-), Q1.3 (E), R54.2, R58.2, U26.12 (GND), X1.2 (GND), X2.7 (GND)
- net IPL0: now also U2.8.22 (IO22)
- net IPL1: now also U2.8.21 (IO21)
- net IPL2: now also U2.8.20 (I020)
- net IRQ1: now also J10.5b (Pin_5b), U2.8.7 (I7), U32.11 (I1); no longer J10.6b (Pin_6b)
- net IRQ2: now also J10.6b (Pin_6b), U2.8.8 (I8), U32.12 (I2); no longer J10.7b (Pin_7b)
- net IRQ3: now also J10.7b (Pin_7b), U2.8.9 (I9), U32.13 (I3); no longer J10.8b (Pin_8b)
- net IRQ6: now also J10.8b (Pin_8b), U2.8.10 (I10), U32.3 (I6); no longer J10.11b (Pin_11b)
- net RESET: no longer R50.2
- net /IO_CS: now also U2.7.4 (E1)
- net /RD: now also U2.9.22 (~{RD}), U26.2 (/RD)
- net /RESET: now also R50.2
- net at U2.2_C1.1, U2.3_C1.1, U2.4_C1.1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: now also U2.7_C1.1, U2.8_C1.1, U2.9_C1.1, U3.0_C1.1
- net at U2.2_C1.2, U2.3_C1.2, U2.4_C1.2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: now also U2.7_C1.2, U2.8_C1.2, U2.9_C1.2, U3.0_C1.2
- net clk_1Mhz: now reaches U2.2.11 (Q3)
- net clk_1Mhz: now also U2.9.15 (CLK1), U2.9.18 (CLK2), U2.9.9 (CLK0)
- net IRQ4 renamed IACK1
- net IACK1: now also U2.8.19 (IO19), U30.14 (O1)
- net IRQ5 renamed IACK2
- net IACK2: now also U2.8.18 (IO18), U30.13 (O2)
- net IRQ7 renamed IACK6
- net IACK6: now also U2.8.16 (IO16), U30.9 (O6)
- net /RAM_CS: no longer names the net of U2.6.2
- net /ROM_CE: no longer names the net of U2.6.1
- new net: U32.10 (IO), U32.14 (GS), U32.15 (EO), U32.5 (EI), U32.8 (GND)
- new net: U2.8.23 (I23), U32.6 (S2)
- new net: U2.8.14 (I14), U32.7 (S1)
- new net: U2.8.13 (I13), U32.9 (S0)
- new net: D9.2 (A), Q1.2 (B), R58.1
- new net: D9.1 (K), R57.2
- new net: Q1.1 (C), R56.2
- new net: BT1.1 (+), D7.2 (A), R55.1
- new net: D7.1 (K), D8.1 (K), Q2.1 (C), R55.2, U26.24 (VCC)
- new net: R53.2, R54.1, U26.23 (PWR_DOWN)
- new net: Q2.2 (B), R56.1
- new net: U30.4 (E1), U31.7 (O7)
- new net: U31.4 (E1), U31.5 (E2), U31.8 (GND)
- new net 32khz: U26.10 (OSC_IN), X2.8 (OUT)
- new net IACK3: J10.11b (Pin_11b), U2.8.17 (IO17), U30.12 (O3)
- new net IACK4: U30.11 (O4)
- new net IACK5: U30.10 (O5)
- new net IACK7: U30.7 (O7)
- new net RTC: U2.7.9 (O6), U26.1 (/CS)
- new net TIMER: U2.7.10 (O5)
- now unconnected: U2.6.3
- no-connect marks 6 -> 11
Other:
- note added: "TIMER = 0x4500 RTC = 0x4600"
- note removed: "PARA FINS DE TESTE NO LUGAR DE /ROM_CE E /RAM_CS ESTOU USANDO O SINAL DA CPU /AS"
- note removed: "nao estou usando o chip que pode provocar wait states nesse momento DTACK está sendo tratado na GAL"
- moved on the sheet: CU21_C2, D4, D5, D6, J10, R23, R24, R25, R33, R34, R35, R36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

Commit message: Interrupts working update...
Parts:
- removed U30, U31: 74LS138, symbol 74xx:74LS138
- removed X2: 32KHZ, Oscillator:Oscillator_DIP-14, symbol Oscillator:ACO-xxxMHz-A
Connections:
- net +5V: now also U2.6.4
- net IRQ6: now also U2.5.5, U2.6.6
- net at U32.10 (IO), U32.14 (GS), U32.15 (EO)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: now also U2.8.12 (GND)
- net at U2.6.8: no longer U2.6.4
- no-connect marks 11 -> 9
Other:
- moved on the sheet: U32

Commit message: update...
Connections:
- net C.E: no longer J10.19b (Pin_19b)
- net C.R/W: no longer U2.9.23 (~{WR})
- net /RD: no longer U2.9.22 (~{RD})
- net /RDL: now reaches J10.28b (Pin_28b)
- net /RDL: now also U2.9.22 (~{RD})
- new net /WRL: J10.19b (Pin_19b), U2.9.23 (~{WR})
Changed lines of the file:
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@@
-    (stroke (width 0) (type default))
-  )
-  (bus_entry (at 331.47 87.63) (size -2.54 2.54)
     (stroke (width 0) (type default))
   )
@@
     (stroke (width 0) (type default))
   )
-  (wire (pts (xy 328.93 90.17) (xy 307.34 90.17))
-    (stroke (width 0) (type default))
-  )
   (wire (pts (xy 334.01 100.33) (xy 350.52 100.33))
     (stroke (width 0) (type default))
@@
     (stroke (width 0) (type default))
   )
+  (wire (pts (xy 320.04 90.17) (xy 307.34 90.17))
+    (stroke (width 0) (type default))
+  )
   (wire (pts (xy 64.77 198.12) (xy 46.99 198.12))
     (stroke (width 0) (type default))
@@
     (stroke (width 0) (type default))
   )
-  (bus (pts (xy 331.47 87.63) (xy 331.47 90.17))
-    (stroke (width 0) (type default))
-  )
   (bus (pts (xy 257.81 224.79) (xy 276.86 224.79))
     (stroke (width 0) (type default))
@@
     (stroke (width 0) (type default))
   )
-  (wire (pts (xy 344.17 120.65) (xy 350.52 120.65))
+  (wire (pts (xy 340.36 120.65) (xy 350.52 120.65))
     (stroke (width 0) (type default))
   )
@@
     (stroke (width 0) (type default))
   )
-  (wire (pts (xy 344.17 118.11) (xy 350.52 118.11))
+  (wire (pts (xy 318.77 113.03) (xy 307.34 113.03))
+    (stroke (width 0) (type default))
+  )
+  (wire (pts (xy 340.36 118.11) (xy 350.52 118.11))
     (stroke (width 0) (type default))
   )
@@
     (stroke (width 0) (type default))
   )
-  (bus (pts (xy 331.47 80.01) (xy 331.47 87.63))
+  (bus (pts (xy 331.47 80.01) (xy 331.47 90.17))
     (stroke (width 0) (type default))
   )
@@
     (effects (font (size 1.27 1.27)) (justify left bottom))
   )
-  (label "D2" (at 344.17 36.83 0)
+  (label "D2" (at 344.17 36.83 0) (fields_autoplaced)
     (effects (font (size 1.27 1.27)) (justify left bottom))
   )
@@
   )
   (label "A1" (at 372.11 44.45 0) (fields_autoplaced)
-    (effects (font (size 1.27 1.27)) (justify left bottom))
-  )
-  (label "C.E" (at 307.34 90.17 0) (fields_autoplaced)
     (effects (font (size 1.27 1.27)) (justify left bottom))
   )
@@
     (effects (font (size 1.27 1.27)) (justify left bottom))
   )
-  (label "D1" (at 344.17 34.29 0)
+  (label "D1" (at 344.17 34.29 0) (fields_autoplaced)
     (effects (font (size 1.27 1.27)) (justify left bottom))
   )
@@
   (label "A19" (at 247.65 90.17 0) (fields_autoplaced)
     (effects (font (size 1.27 1.27)) (justify left bottom))
-  )
-  (label "{slash}RD" (at 344.17 118.11 180) (fields_autoplaced)
-    (effects (font (size 1.27 1.27)) (justify right bottom))
   )
   (label "A23" (at 247.65 100.33 0) (fields_autoplaced)
@@
     (effects (font (size 1.27 1.27)) (justify right bottom))
   )
-  (label "D7" (at 344.17 49.53 0)
+  (label "D7" (at 344.17 49.53 0) (fields_autoplaced)
     (effects (font (size 1.27 1.27)) (justify left bottom))
   )
@@
     (effects (font (size 1.27 1.27)) (justify left bottom))
   )
-  (label "D5" (at 344.17 44.45 0)
+  (label "D5" (at 344.17 44.45 0) (fields_autoplaced)
     (effects (font (size 1.27 1.27)) (justify left bottom))
   )
@@
     (effects (font (size 1.27 1.27)) (justify left bottom))
   )
-  (label "D4" (at 344.17 41.91 0)
+  (label "D4" (at 344.17 41.91 0) (fields_autoplaced)
     (effects (font (size 1.27 1.27)) (justify left bottom))
   )
@@
     (effects (font (size 1.27 1.27)) (justify right bottom))
   )
-  (label "D8" (at 344.17 52.07 0)
+  (label "D8" (at 344.17 52.07 0) (fields_autoplaced)
     (effects (font (size 1.27 1.27)) (justify left bottom))
   )
@@
     (effects (font (size 1.27 1.27)) (justify left bottom))
   )
-  (label "C.R{slash}W" (at 344.17 120.65 180) (fields_autoplaced)
-    (effects (font (size 1.27 1.27)) (justify right bottom))
-  )
   (label "A17" (at 247.65 85.09 0) (fields_autoplaced)
     (effects (font (size 1.27 1.27)) (justify left bottom))
@@
     (effects (font (size 1.27 1.27)) (justify left bottom))
   )
-  (label "D6" (at 344.17 46.99 0)
+  (label "D6" (at 344.17 46.99 0) (fields_autoplaced)
     (effects (font (size 1.27 1.27)) (justify left bottom))
   )
@@
     (effects (font (size 1.27 1.27)) (justify left bottom))
   )
-  (label "D3" (at 344.17 39.37 0)
+  (label "D3" (at 344.17 39.37 0) (fields_autoplaced)
     (effects (font (size 1.27 1.27)) (justify left bottom))
   )
@@
   (label "A1" (at 274.32 165.1 0) (fields_autoplaced)
     (effects (font (size 1.27 1.27)) (justify left bottom))
+  )
+  (global_label "{slash}WRL" (shape input) (at 320.04 90.17 0) (fields_autoplaced)
+    (effects (font (size 1.27 1.27)) (justify left))
+    (property "Intersheetrefs" "${INTERSHEET_REFS}" (at 328.1052 90.17 0)
+      (effects (font (size 1.27 1.27)) (justify left) hide)
+    )
   )
   (global_label "key_cs" (shape input) (at 309.88 123.19 0) (fields_autoplaced)
@@
     )
   )
+  (global_label "{slash}RDL" (shape input) (at 340.36 118.11 180) (fields_autoplaced)
+    (effects (font (size 1.27 1.27)) (justify right))
+    (property "Intersheetrefs" "${INTERSHEET_REFS}" (at 332.4762 118.11 0)
+      (effects (font (size 1.27 1.27)) (justify right) hide)
+    )
+  )
   (global_label "{slash}IO_CS" (shape input) (at 345.44 177.8 180) (fields_autoplaced)
     (effects (font (size 1.27 1.27)) (justify right))
@@
     )
   )
+  (global_label "{slash}RDL" (shape input) (at 318.77 113.03 0) (fields_autoplaced)
+    (effects (font (size 1.27 1.27)) (justify left))
+    (property "Intersheetrefs" "${INTERSHEET_REFS}" (at 326.6538 113.03 0)
+      (effects (font (size 1.27 1.27)) (justify left) hide)
+    )
+  )
   (global_label "RESET" (shape input) (at 309.88 133.35 0) (fields_autoplaced)
     (effects (font (size 1.27 1.27)) (justify left))
@@
     )
   )
+  (global_label "{slash}WRL" (shape input) (at 340.36 120.65 180) (fields_autoplaced)
+    (effects (font (size 1.27 1.27)) (justify right))
+    (property "Intersheetrefs" "${INTERSHEET_REFS}" (at 332.2948 120.65 0)
+      (effects (font (size 1.27 1.27)) (justify right) hide)
+    )
+  )

Commit message: Atmega8 code completed
Parts:
- added R59, R60, R61, R62: 4K7, Resistor_THT:R_Axial_DIN0204_L3.6mm_D1.6mm_P5.08mm_Horizontal, symbol Device:R
- added U2.3: 74LS138, symbol 74xx:74LS138
- added U3.2: 74LS74, symbol 74xx:74LS74
- added U31: ATmega8-16P, Package_DIP:DIP-28_W7.62mm, symbol MCU_Microchip_ATmega:ATmega8-16P
- renumbered U32 to U3.1
Connections:
- net +5V: now also R59.1, R60.1, R61.1, R62.1, U3.2.2 (D), U3.2.3 (C)
- net A1: no longer U2.8.3 (I3)
- net A2: no longer U2.8.2 (I2)
- net A3: no longer U2.8.1 (I1)
- net C.FC0: now also U2.3.1 (A0); no longer U2.8.4 (I4)
- net C.FC1: now also U2.3.2 (A1); no longer U2.8.5 (I5)
- net C.FC2: now also U2.3.3 (A2); no longer U2.8.6 (I6)
- net C./AS: now also U2.3.4 (E1), U2.3.5 (E2)
- net C./VPA: now also U3.2.4 (~{S}); no longer U2.8.15 (IO15)
- net IACK1: no longer J10.9b (Pin_9b), U2.8.19 (IO19)
- net IACK2: no longer J10.10b (Pin_10b), U2.8.18 (IO18)
- net IACK3: no longer J10.11b (Pin_11b), U2.8.17 (IO17)
- net IACK6: now also U2.3.7 (O7); no longer J10.12b (Pin_12b), U2.8.16 (IO16)
- net IPL0: now also U31.23 (PC0); no longer U2.8.22 (IO22)
- net IPL1: now also U31.24 (PC1); no longer U2.8.21 (IO21)
- net IPL2: now also U31.25 (PC2); no longer U2.8.20 (I020)
- net IRQ1: now also R61.2, U31.4 (PD2); no longer U2.8.7 (I7)
- net IRQ2: now also R60.2, U31.5 (PD3); no longer U2.8.8 (I8)
- net IRQ3: now also R59.2, U31.6 (PD4); no longer U2.8.9 (I9)
- net IRQ6: now also R62.2, U3.2.5 (Q); no longer U2.5.5, U2.6.6, U2.8.10 (I10)
- net at U3.1.10 (IO), U3.1.14 (GS), U3.1.15 (EO)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: no longer U2.8.12 (GND)
- net at U2.8.23 (I23): no longer U3.1.6 (S2)
- net at U2.8.14 (I14): no longer U3.1.7 (S1)
- net at U2.8.13 (I13): no longer U3.1.9 (S0)
- net at U2.9.10 (OUT0): now also U3.2.1 (~{R})
- new net: U2.3.16 (VCC), U2.3.6 (E3)
- new net C.IPL0: U3.1.9 (S0)
- new net C.IPL1: U3.1.7 (S1)
- new net C.IPL2: U3.1.6 (S2)
- new net FC0: U31.16 (PB2)
- new net FC1: U31.17 (PB3)
- new net FC2: U31.18 (PB4)
- new net IRQ4: U31.11 (PD5)
- new net IRQ5: U31.12 (PD6)
- new net IRQ7: U31.13 (PD7)
- new net Ligar Irq3 por exemplo: U2.5.5, U2.6.6
- new net VPA: U31.28 (PC5)
Other:
- note added: "A0"
- note added: "A1"
- note added: "A5"
- note added: "D0"
- note added: "D1"
- note added: "D10"
- note added: "D11"
- note added: "D12"
- note added: "D13"
- note added: "D2"
- note added: "D3"
- note added: "D4"
- note added: "D5"
- note added: "D6"
- note added: "D7"
- note added: "D8"
- note added: "D9"
- note added: "cortei o resistor reconectar"
- moved on the sheet: U2.8

Commit message: Atmega8 firmware and schematics, ints working
Parts:
- removed R59, R60, R61, R62: 4K7, Resistor_THT:R_Axial_DIN0204_L3.6mm_D1.6mm_P5.08mm_Horizontal, symbol Device:R
- removed U2.8: PAL20L8, symbol Logic_Programmable:PAL20L8
- removed U3.1: 74LS148, symbol 74xx:74LS148
Connections:
- net IRQ2: now also U31.15 (PB1)
- net /RESET: no longer R32.2, U2.1.17 (HALT), U2.5.4, U2.5.9
- net FC0: no longer names the net of U31.16 (PB2)
- net FC1: no longer names the net of U31.17 (PB3)
- net FC2: no longer names the net of U31.18 (PB4)
- net IACK6 renamed /VPA
- net VPA: no longer names the net of U31.28 (PC5)
- new net /HALT: R32.2, U2.1.17 (HALT), U2.5.4, U2.5.9
Other:
- note added: "1KHZ"
- note added: "D"
- moved on the sheet: R49, R50, R51, R52, SW3, U2.5C, U2.5E, U2.5F, U2.6B, U2.6C, U2.7, U31
