File: schematics/MC68000/cpuNoBuffer.kicad_sch (KiCad schematic)
At the start: 71 parts, among them J10 Conn_02x37_Row_Letter_Last, Q1 NPN, Q2 PNP, SW2 Reset, SW3 Xmodem, U2.1 68000D, U2.2 74LS161, U2.2_C1 100nF, U2.3 74LS138, U2.3_C1 100nF, U2.4 ICM7555xB, U2.4_C1 100nF, U2.5 74LS05, U2.5_C1 100nF, U2.6 74LS00, U2.6_C1 100nF, U2.7 74LS138, U2.7_C1 100nF, U2.8_C1 100nF, U2.9 8253, U2.9_C1 100nF, U21_C1 100nF, U3.0_C1 100nF, U3.2 74LS74, U31 ATmega8-16P, X1 16MHZ

Commit message: Update
Parts:
- removed U3.2: 74LS74, symbol 74xx:74LS74
- renumbered U31 to U2.8, U26 to U3.0
Changed lines of the file:
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@@
   (junction (at 378.46 15.24) (diameter 0) (color 0 0 0 0)
   )
-  (junction (at 379.73 113.03) (diameter 0) (color 0 0 0 0)
-  )
   (junction (at 90.17 30.48) (diameter 0) (color 0 0 0 0)
   )
@@
     (stroke (width 0) (type default))
   )
-  (wire (pts (xy 370.84 102.87) (xy 391.16 102.87))
-    (stroke (width 0) (type default))
-  )
   (wire (pts (xy 151.13 53.34) (xy 152.4 54.61))
     (stroke (width 0) (type default))
@@
     (stroke (width 0) (type default))
   )
-  (wire (pts (xy 391.16 120.65) (xy 391.16 128.27))
-    (stroke (width 0) (type default))
-  )
   (wire (pts (xy 158.75 233.68) (xy 152.4 233.68))
     (stroke (width 0) (type default))
@@
     (stroke (width 0) (type default))
   )
-  (wire (pts (xy 379.73 113.03) (xy 379.73 115.57))
-    (stroke (width 0) (type default))
-  )
   (wire (pts (xy 222.25 24.13) (xy 224.79 24.13))
     (stroke (width 0) (type default))
@@
     (stroke (width 0) (type default))
   )
-  (wire (pts (xy 379.73 110.49) (xy 379.73 113.03))
-    (stroke (width 0) (type default))
-  )
   (wire (pts (xy 195.58 41.91) (xy 195.58 52.07))
     (stroke (width 0) (type default))
@@
     (stroke (width 0) (type default))
   )
-  (wire (pts (xy 379.73 113.03) (xy 383.54 113.03))
-    (stroke (width 0) (type default))
-  )
   (bus (pts (xy 257.81 140.97) (xy 257.81 143.51))
     (stroke (width 0) (type default))
@@
     (stroke (width 0) (type default))
   )
-  (wire (pts (xy 401.32 115.57) (xy 398.78 115.57))
-    (stroke (width 0) (type default))
-  )
   (wire (pts (xy 287.02 227.33) (xy 295.91 227.33))
     (stroke (width 0) (type default))
@@
     (stroke (width 0) (type default))
   )
-  (wire (pts (xy 391.16 128.27) (xy 392.43 128.27))
-    (stroke (width 0) (type default))
-  )
   (bus (pts (xy 335.28 36.83) (xy 335.28 39.37))
     (stroke (width 0) (type default))
@@
     (stroke (width 0) (type default))
   )
-  (wire (pts (xy 379.73 115.57) (xy 383.54 115.57))
-    (stroke (width 0) (type default))
-  )
   (wire (pts (xy 307.34 49.53) (xy 323.85 49.53))
     (stroke (width 0) (type default))
@@
     (stroke (width 0) (type default))
   )
-  (wire (pts (xy 391.16 102.87) (xy 391.16 105.41))
-    (stroke (width 0) (type default))
-  )
   (wire (pts (xy 276.86 185.42) (xy 283.21 185.42))
     (stroke (width 0) (type default))
@@
     (effects (font (size 1.27 1.27)) (justify left bottom))
   )
-  (label "C.{slash}VPA" (at 392.43 128.27 0) (fields_autoplaced)
-    (effects (font (size 1.27 1.27)) (justify left bottom))
-  )
   (label "A15" (at 247.65 80.01 0) (fields_autoplaced)
     (effects (font (size 1.27 1.27)) (justify left bottom))
@@
     (effects (font (size 1.27 1.27)) (justify right bottom))
   )
-  (label "IRQ6" (at 401.32 115.57 0) (fields_autoplaced)
-    (effects (font (size 1.27 1.27)) (justify left bottom))
-  )
   (label "D14" (at 283.21 133.35 0) (fields_autoplaced)
     (effects (font (size 1.27 1.27)) (justify left bottom))
@@
   (symbol (lib_id "MCU_Microchip_ATmega:ATmega8-16P") (at 359.41 191.77 0) (unit 1)
     (in_bom yes) (on_board yes) (dnp no) (fields_autoplaced)
-    (property "Reference" "U31" (at 364.1441 153.67 0)
+    (property "Reference" "U2.8" (at 364.1441 153.67 0)
       (effects (font (size 1.27 1.27)) (justify left))
     )
@@
       (project "MC68000"
         (path "/99c9748a-87b3-41bd-bdc2-3a5f137c7a40/cb1c4173-bc78-475d-9381-bcb9d50be77b"
-          (reference "U31") (unit 1)
-        )
-      )
-    )
-  )
-  (symbol (lib_id "power:+5V") (at 379.73 110.49 0) (unit 1)
-    (in_bom yes) (on_board yes) (dnp no) (fields_autoplaced)
-    (property "Reference" "#PWR066" (at 379.73 114.3 0)
-      (effects (font (size 1.27 1.27)) hide)
-    )
-    (property "Value" "+5V" (at 379.73 105.41 0)
-      (effects (font (size 1.27 1.27)))
-    )
-    (property "Footprint" "" (at 379.73 110.49 0)
-      (effects (font (size 1.27 1.27)) hide)
-    )
-    (property "Datasheet" "" (at 379.73 110.49 0)
-      (effects (font (size 1.27 1.27)) hide)
-    )
-    (pin "1")
-    (instances
-      (project "MC68000"
-        (path "/99c9748a-87b3-41bd-bdc2-3a5f137c7a40/cb1c4173-bc78-475d-9381-bcb9d50be77b"
-          (reference "#PWR066") (unit 1)
+          (reference "U2.8") (unit 1)
         )
       )
@@
   (symbol (lib_id "OSLIB:MM58167") (at 353.06 29.21 0) (unit 1)
     (in_bom yes) (on_board yes) (dnp no) (fields_autoplaced)
-    (property "Reference" "U26" (at 362.8741 27.94 0)
+    (property "Reference" "U3.0" (at 362.8741 27.94 0)
       (effects (font (size 1.27 1.27)) (justify left))
     )
@@
       (project "MC68000"
         (path "/99c9748a-87b3-41bd-bdc2-3a5f137c7a40/cb1c4173-bc78-475d-9381-bcb9d50be77b"
-          (reference "U26") (unit 1)
+          (reference "U3.0") (unit 1)
         )
       )
@@
     )
   )
-  (symbol (lib_id "74xx:74LS74") (at 52.07 232.41 0) (unit 2)
-    (in_bom yes) (on_board yes) (dnp no) (fields_autoplaced)
-    (property "Reference" "U3.2" (at 54.2641 222.25 0)
-      (effects (font (size 1.27 1.27)) (justify left))
-    )
-    (property "Value" "74LS74" (at 54.2641 224.79 0)
-      (effects (font (size 1.27 1.27)) (justify left))
-    )
-    (property "Footprint" "" (at 52.07 232.41 0)
-      (effects (font (size 1.27 1.27)) hide)
-    )
-    (property "Datasheet" "74xx/74hc_hct74.pdf" (at 52.07 232.41 0)
-      (effects (font (size 1.27 1.27)) hide)
-    )
-    (pin "6")
-    (pin "10")
-    (pin "4")
-    (pin "1")
-    (pin "2")
-    (pin "3")
-    (pin "11")
-    (pin "8")
-    (pin "9")
-    (pin "12")
-    (pin "13")
-    (pin "7")
-    (pin "14")
-    (pin "5")
-    (instances
-      (project "MC68000"
-        (path "/99c9748a-87b3-41bd-bdc2-3a5f137c7a40/cb1c4173-bc78-475d-9381-bcb9d50be77b"
-          (reference "U3.2") (unit 2)
-        )
-      )
-    )
-  )
   (symbol (lib_id "power:+5V") (at 93.98 97.79 0) (unit 1)
     (in_bom yes) (on_board yes) (dnp no) (fields_autoplaced)
@@
     )
   )
-  (symbol (lib_id "74xx:74LS74") (at 391.16 113.03 0) (mirror x) (unit 1)
-    (in_bom yes) (on_board yes) (dnp no)
-    (property "Reference" "U3.2" (at 393.3541 123.19 0)
-      (effects (font (size 1.27 1.27)) (justify left))
-    )
-    (property "Value" "74LS74" (at 393.3541 120.65 0)
-      (effects (font (size 1.27 1.27)) (justify left))
-    )
-    (property "Footprint" "" (at 391.16 113.03 0)
-      (effects (font (size 1.27 1.27)) hide)
-    )
-    (property "Datasheet" "74xx/74hc_hct74.pdf" (at 391.16 113.03 0)
-      (effects (font (size 1.27 1.27)) hide)
-    )
-    (pin "6")
-    (pin "10")
-    (pin "4")
-    (pin "1")
-    (pin "2")
-    (pin "3")
-    (pin "11")
-    (pin "8")
-    (pin "9")
-    (pin "12")
-    (pin "13")
-    (pin "7")
-    (pin "14")
-    (pin "5")
-    (instances
-      (project "MC68000"
-        (path "/99c9748a-87b3-41bd-bdc2-3a5f137c7a40/cb1c4173-bc78-475d-9381-bcb9d50be77b"
-          (reference "U3.2") (unit 1)
-        )
-      )
-    )
-  )
   (symbol (lib_id "74xx:74LS05") (at 72.39 198.12 180) (unit 4)
     (in_bom yes) (on_board yes) (dnp no) (fields_autoplaced)
@@
         )
       )
-    )
-  )
-  (symbol (lib_id "74xx:74LS74") (at 74.93 232.41 0) (unit 3)
-    (in_bom yes) (on_board yes) (dnp no) (fields_autoplaced)
-    (property "Reference" "U3.2" (at 81.28 231.14 0)
-      (effects (font (size 1.27 1.27)) (justify left))
-    )
-    (property "Value" "74LS74" (at 81.28 233.68 0)
-      (effects (font (size 1.27 1.27)) (justify left))
-    )
-    (property "Footprint" "" (at 74.93 232.41 0)
-      (effects (font (size 1.27 1.27)) hide)
-    )
-    (property "Datasheet" "74xx/74hc_hct74.pdf" (at 74.93 232.41 0)
-      (effects (font (size 1.27 1.27)) hide)
-    )
-    (pin "6")
-    (pin "10")
-    (pin "4")
-    (pin "1")
-    (pin "2")
-    (pin "3")
-    (pin "11")
-    (pin "8")
-    (pin "9")
-    (pin "12")
-    (pin "13")
-    (pin "7")
-    (pin "14")
-    (pin "5")
-    (instances
-      (project "MC68000"
-        (path "/99c9748a-87b3-41bd-bdc2-3a5f137c7a40/cb1c4173-bc78-475d-9381-bcb9d50be77b"
-          (reference "U3.2") (unit 3)
-        )
-      )
