File: schematics/MC68000/cpuNoBuffer.kicad_sch (KiCad schematic)
At the start: 70 parts, among them J10 Conn_02x37_Row_Letter_Last, Q1 NPN, Q2 PNP, SW2 Reset, SW3 Xmodem, U2.1 68000D, U2.2 74LS161, U2.2_C1 100nF, U2.3 74LS138, U2.3_C1 100nF, U2.4 ICM7555xB, U2.4_C1 100nF, U2.5 74LS05, U2.5_C1 100nF, U2.6 74LS00, U2.6_C1 100nF, U2.7 74LS138, U2.7_C1 100nF, U2.8 ATmega8-16P, U2.8_C1 100nF, U2.9 8253, U2.9_C1 100nF, U21_C1 100nF, U3.0_C1 100nF, X1 16MHZ

Commit message: tinyBasic running
Connections:
- net TIMER is gone; now on net RTC_CS: U2.7.10 (O5)
- net D0: now also U2.9.8 (D0), U3.0.15 (D0)
- net D1: now also U2.9.7 (D1), U3.0.16 (D1); no longer U2.9.8 (D0), U3.0.15 (D0)
- net D2: now also U2.9.6 (D2), U3.0.17 (D2); no longer U2.9.7 (D1), U3.0.16 (D1)
- net D3: now also U2.9.5 (D3), U3.0.18 (D3); no longer U2.9.6 (D2), U3.0.17 (D2)
- net D4: now also U2.9.4 (D4), U3.0.19 (D4); no longer U2.9.5 (D3), U3.0.18 (D3)
- net D5: now also U2.9.3 (D5), U3.0.20 (D5); no longer U2.9.4 (D4), U3.0.19 (D4)
- net D6: now also U2.9.2 (D6), U3.0.21 (D6); no longer U2.9.3 (D5), U3.0.20 (D5)
- net D7: now also U2.9.1 (D7), U3.0.22 (D7); no longer U2.9.2 (D6), U3.0.21 (D6)
- net D8: no longer U2.9.1 (D7), U3.0.22 (D7)
- net TIMER_CS: now reaches U2.9.21 (~{CS})
- net TIMER_CS: now also U2.7.9 (O6)
- net RTC renamed RTC_CS
- net RTC_CS: no longer U2.7.9 (O6)
Other:
- note added: "RTC = 0x4500 TIMER = 0x4600"
- note removed: "TIMER = 0x4500 RTC = 0x4600"

Commit message: updating...
Parts:
- renumbered U2.3 to U3.2

Commit message: updating...
Connections:
- net C.FC0: no longer U3.2.1 (A0)
- net C.FC1: no longer U3.2.2 (A1)
- net C.FC2: no longer U3.2.3 (A2)
- new net FC0: U3.2.1 (A0)
- new net FC1: U3.2.2 (A1)
- new net FC2: U3.2.3 (A2)
Changed lines of the file:
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@@
 		)
 	)
-	(label "C.FC2"
+	(label "FC2"
 		(at 274.32 172.72 0)
 		(effects
@@
 		)
 	)
-	(label "C.FC0"
+	(label "FC0"
 		(at 274.32 167.64 0)
 		(effects
@@
 		)
 	)
-	(label "C.FC1"
+	(label "FC1"
 		(at 274.32 170.18 0)
 		(effects

Commit message: updating...
Connections:
- net C./AS: no longer U3.2.4 (E1), U3.2.5 (E2)
- net C./VPA: no longer R35.2, U2.1.21 (VPA)
- net /VPA: now also R35.2, U2.1.21 (VPA)
- net at U3.2.8 (GND): now also U3.2.4 (E1), U3.2.5 (E2)
Changed lines of the file:
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@@
 	)
 	(junction
-		(at 276.86 182.88)
-		(diameter 0)
-		(color 0 0 0 0)
-	)
-	(junction
 		(at 130.81 279.4)
 		(diameter 0)
@@
 	)
 	(junction
+		(at 276.86 185.42)
+		(diameter 0)
+		(color 0 0 0 0)
+	)
+	(junction
 		(at 30.48 127)
 		(diameter 0)
@@
 	(wire
 		(pts
-			(xy 260.35 182.88) (xy 276.86 182.88)
+			(xy 53.34 55.88) (xy 71.12 55.88)
 		)
 		(stroke
@@
 	(wire
 		(pts
-			(xy 53.34 55.88) (xy 71.12 55.88)
+			(xy 180.34 24.13) (xy 185.42 24.13)
 		)
 		(stroke
@@
 	(wire
 		(pts
-			(xy 180.34 24.13) (xy 185.42 24.13)
+			(xy 328.93 97.79) (xy 307.34 97.79)
 		)
 		(stroke
@@
 	(wire
 		(pts
-			(xy 328.93 97.79) (xy 307.34 97.79)
+			(xy 295.91 193.04) (xy 295.91 196.85)
 		)
 		(stroke
@@
 	(wire
 		(pts
+			(xy 276.86 196.85) (xy 276.86 185.42)
+		)
+		(stroke
+			(width 0)
+			(type default)
+		)
+	)
+	(wire
+		(pts
 			(xy 73.66 279.4) (xy 73.66 271.78)
 		)
@@
 		)
 	)
+	(wire
+		(pts
+			(xy 295.91 196.85) (xy 276.86 196.85)
+		)
+		(stroke
+			(width 0)
+			(type default)
+		)
+	)
 	(bus
 		(pts
@@
 		)
 	)
-	(label "C.{slash}VPA"
+	(label "{slash}VPA"
 		(at 163.83 92.71 0)
 		(effects
@@
 		(effects
 			(font
-				(size 1.27 1.27)
-			)
-			(justify left bottom)
-		)
-	)
-	(label "C.{slash}AS"
-		(at 274.32 182.88 0)
-		(effects
-			(font

Commit message: updating...
Connections:
- net FC0: now also U2.8.16 (PB2)
- net FC1: now also U2.8.17 (PB3)
- net FC2: now also U2.8.18 (PB4)
Changed lines of the file:
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@@
 		)
 	)
+	(wire
+		(pts
+			(xy 384.81 171.45) (xy 374.65 171.45)
+		)
+		(stroke
+			(width 0)
+			(type default)
+		)
+	)
 	(bus
 		(pts
@@
 	(wire
 		(pts
+			(xy 384.81 173.99) (xy 374.65 173.99)
+		)
+		(stroke
+			(width 0)
+			(type default)
+		)
+	)
+	(wire
+		(pts
 			(xy 73.66 254) (xy 86.36 254)
 		)
@@
 	(wire
 		(pts
+			(xy 384.81 168.91) (xy 374.65 168.91)
+		)
+		(stroke
+			(width 0)
+			(type default)
+		)
+	)
+	(wire
+		(pts
 			(xy 276.86 185.42) (xy 283.21 185.42)
 		)
@@
 		)
 	)
+	(label "FC2"
+		(at 384.81 173.99 0)
+		(effects
+			(font
+				(size 1.27 1.27)
+			)
+			(justify left bottom)
+		)
+	)
 	(label "D1"
 		(at 347.98 97.79 0)
@@
 		(effects
 			(font
+				(size 1.27 1.27)
+			)
+			(justify left bottom)
+		)
+	)
+	(label "FC0"
+		(at 384.81 168.91 0)
+		(effects
+			(font
+				(size 1.27 1.27)
+			)
+			(justify left bottom)
+		)
+	)
+	(label "FC1"
+		(at 384.81 171.45 0)
+		(effects
+			(font

Commit message: updating...
Connections:
- net IRQ2: no longer U2.8.15 (PB1)
- net IRQ7: now also U2.8.15 (PB1)
Changed lines of the file:
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@@
 		)
 	)
-	(wire
-		(pts
-			(xy 374.65 207.01) (xy 381 207.01)
-		)
-		(stroke
-			(width 0)
-			(type default)
-		)
-	)
 	(bus
 		(pts
@@
 	(wire
 		(pts
+			(xy 374.65 217.17) (xy 381 217.17)
+		)
+		(stroke
+			(width 0)
+			(type default)
+		)
+	)
+	(wire
+		(pts
 			(xy 99.06 254) (xy 109.22 254)
 		)
@@
 	(wire
 		(pts
-			(xy 381 166.37) (xy 381 207.01)
+			(xy 381 166.37) (xy 381 217.17)
 		)
 		(stroke

Commit message: updating...
Parts:
- added D10: Sys Alive, Diode_THT:D_DO-34_SOD68_P5.08mm_Vertical_AnodeUp, symbol Device:LED
- added R59: 470R, Resistor_THT:R_Axial_DIN0204_L3.6mm_D1.6mm_P5.08mm_Horizontal, symbol Device:R
Connections:
- net at U2.8.19 (PB5): now also D10.2 (A)
- net at U2.8.7 (VCC): now also R59.2
- new net: D10.1 (K), R59.1
Changed lines of the file:
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@@
 	(wire
 		(pts
+			(xy 374.65 176.53) (xy 393.7 176.53)
+		)
+		(stroke
+			(width 0)
+			(type default)
+		)
+	)
+	(wire
+		(pts
 			(xy 389.89 67.31) (xy 392.43 67.31)
 		)
@@
 		)
 	)
+	(wire
+		(pts
+			(xy 400.05 167.64) (xy 400.05 171.45)
+		)
+		(stroke
+			(width 0)
+			(type default)
+		)
+	)
 	(bus
 		(pts
@@
 		)
 	)
+	(wire
+		(pts
+			(xy 393.7 179.07) (xy 400.05 179.07)
+		)
+		(stroke
+			(width 0)
+			(type default)
+		)
+	)
 	(bus
 		(pts
@@
 	(wire
 		(pts
+			(xy 359.41 156.21) (xy 359.41 149.86)
+		)
+		(stroke
+			(width 0)
+			(type default)
+		)
+	)
+	(wire
+		(pts
 			(xy 370.84 97.79) (xy 374.65 97.79)
 		)
@@
 	(wire
 		(pts
+			(xy 393.7 176.53) (xy 393.7 179.07)
+		)
+		(stroke
+			(width 0)
+			(type default)
+		)
+	)
+	(wire
+		(pts
 			(xy 46.99 184.15) (xy 54.61 184.15)
 		)
@@
 	(wire
 		(pts
+			(xy 359.41 149.86) (xy 400.05 149.86)
+		)
+		(stroke
+			(width 0)
+			(type default)
+		)
+	)
+	(wire
+		(pts
 			(xy 307.34 49.53) (xy 323.85 49.53)
 		)
@@
 	(wire
 		(pts
+			(xy 400.05 149.86) (xy 400.05 160.02)
+		)
+		(stroke
+			(width 0)
+			(type default)
+		)
+	)
+	(wire
+		(pts
 			(xy 288.29 218.44) (xy 288.29 220.98)
 		)
@@
 	)
 	(symbol
+		(lib_id "Device:LED")
+		(at 400.05 175.26 270)
+		(unit 1)
+		(exclude_from_sim no)
+		(in_bom yes)
+		(on_board yes)
+		(dnp no)
+		(property "Reference" "D10"
+			(at 402.59 172.4024 90)
+			(effects
+				(font
+					(size 1.27 1.27)
+				)
+				(justify left)
+			)
+		)
+		(property "Value" "Sys Alive"
+			(at 396.748 180.848 90)
+			(effects
+				(font
+					(size 1.27 1.27)
+				)
+				(justify left)
+			)
+		)
+		(property "Footprint" "Diode_THT:D_DO-34_SOD68_P5.08mm_Vertical_AnodeUp"
+			(at 400.05 175.26 0)
+			(effects
+				(font
+					(size 1.27 1.27)
+				)
+				(hide yes)
+			)
+		)
+		(property "Datasheet" "~"
+			(at 400.05 175.26 0)
+			(effects
+				(font
+					(size 1.27 1.27)
+				)
+				(hide yes)
+			)
+		)
+		(property "Description" ""
+			(at 400.05 175.26 0)
+			(effects
+				(font
+					(size 1.27 1.27)
+				)
+			)
+		)
+		(pin "1"
+		)
+		(pin "2"
+		)
+		(instances
+			(project "MC68000"
+				(path "/99c9748a-87b3-41bd-bdc2-3a5f137c7a40/cb1c4173-bc78-475d-9381-bcb9d50be77b"
+					(reference "D10")
+					(unit 1)
+				)
+			)
+		)
+	)
+	(symbol
 		(lib_id "power:+5V")
 		(at 39.37 114.3 0)
@@
 				)
 			)
+		)
+	)
+	(symbol
+		(lib_id "Device:R")
+		(at 400.05 163.83 180)
+		(unit 1)
+		(exclude_from_sim no)
+		(in_bom yes)
+		(on_board yes)
+		(dnp no)
+		(property "Reference" "R59"
+			(at 403.86 167.64 0)
+			(effects
+				(font
+					(size 1.27 1.27)
+				)
+				(justify left)
+			)
+		)
+		(property "Value" "470R"
+			(at 402.59 161.29 90)
+			(effects
+				(font
+					(size 1.27 1.27)
+				)
+				(justify left)
+			)
+		)
+		(property "Footprint" "Resistor_THT:R_Axial_DIN0204_L3.6mm_D1.6mm_P5.08mm_Horizontal"
+			(at 401.828 163.83 90)
+			(effects
+				(font
+					(size 1.27 1.27)
+				)
+				(hide yes)
+			)
+		)
+		(property "Datasheet" "~"
+			(at 400.05 163.83 0)
+			(effects
+				(font
+					(size 1.27 1.27)
+				)
+				(hide yes)
+			)
+		)
+		(property "Description" ""
+			(at 400.05 163.83 0)
+			(effects
+				(font
+					(size 1.27 1.27)
+				)
+			)
+		)
+		(pin "1"
+		)
+		(pin "2"
+		)
+		(instances
+			(project "MC68000"
+				(path "/99c9748a-87b3-41bd-bdc2-3a5f137c7a40/cb1c4173-bc78-475d-9381-bcb9d50be77b"
+					(reference "R59")
+					(unit 1)
+				)
+			)

Commit message: inserido comando vga set_txt_color no 68000
Parts:
- renumbered BT1 to BT?, C21 to C?, C20 to C?, C22 to C?, CU21_C2 to CU21_C?, D9 to D?, D4 to D?, D10 to D?, D7 to D?, D8 to D?, D6 to D?, D5 to D?, J10 to J?, JP8 to JP?, JP7 to JP?, JP5 to JP?, JP6 to JP?, Q1 to Q?, Q2 to Q?, R30 to R?, R51 to R?, R58 to R?, R49 to R?, R26 to R?, R35 to R?, R39 to R?, R55 to R?, R29 to R?, R37 to R?, R24 to R?, R32 to R?, R38 to R?, R23 to R?, R34 to R?, R33 to R?, R50 to R?, R56 to R?, R53 to R?, R54 to R?, R59 to R?, R22 to R?, R31 to R?, R36 to R?, R52 to R?, R57 to R?, R40 to R?, R25 to R?, R28 to R?, R27 to R?, SW3 to SW?, SW2 to SW?, U2.2_C1 to U2.2_C?, U2.3_C1 to U2.3_C?, U2.4_C1 to U2.4_C?, U2.5_C1 to U2.5_C?, U2.6_C1 to U2.6_C?, U2.7_C1 to U2.7_C?, U2.8_C1 to U2.8_C?, U2.9_C1 to U2.9_C?, U2.5 to U2.?, U2.8 to U2.?, U2.1 to U2.?, U2.7 to U2.?, U2.4 to U2.?, U2.2 to U2.?, U2.6 to U2.?, U2.9 to U2.?, U21_C1 to U21_C?, U3.0_C1 to U3.0_C?, U3.0 to U3.?, U3.2 to U3.?, X1 to X?
Connections:
- net +5V: now also U2.?.1; no longer U2.?.4
- net C.R/W: now also U2.?.1; no longer U2.?.11
- net Ligar Irq3 por exemplo: now also U2.?.1, U2.?.3; no longer U2.?.5, U2.?.6
- net RESET: now also U2.?.2; no longer U2.?.12
- net SWITCH_OUT: now also U2.?.2; no longer U2.?.6
- net key_cs: now also U2.?.1, U2.?.2; no longer U2.?.10, U2.?.9
- net /HALT: now also U2.?.1, U2.?.2; no longer U2.?.4, U2.?.9
- net /RD: now also U2.?.2; no longer U2.?.10
- net /RESET: now also U2.?.1; no longer U2.?.13
- net at R?.1, SW?.1: now also U2.?.2; no longer U2.?.5
- net at U2.2_C?.1, U2.3_C?.1, U2.4_C?.1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: no longer U2.?.14 (VCC), U2.?.14 (VCC)
- net at U2.2_C?.2, U2.3_C?.2, U2.4_C?.2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: no longer U2.?.7 (GND), U2.?.7 (GND)
- net at U2.?.1, U2.?.3 (Q): now also U2.?.1; no longer U2.?.3
- net at R?.2: now also U2.?.2; no longer U2.?.8
