File: schematics/MC68000/fourUarts.kicad_sch (KiCad schematic)
At the start: 36 parts, among them J3 RS232_1, J4 RS232_1, J5 RS232_1, J6 RS232_1, J7 Conn_02x20_Counter_Clockwise, J8 Conn_02x04_Counter_Clockwise, J9 Conn_02x02_Counter_Clockwise, U18_C1 100nf, U18_C2 100nf, U18_C3 100nf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

Commit message: Ram memory test 2 OK
Changed lines of the file:
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@@
   (symbol (lib_id "Connector_Generic:Conn_02x04_Counter_Clockwise") (at 44.45 140.97 0) (unit 1)
     (in_bom yes) (on_board yes) (dnp no) (fields_autoplaced)
-    (property "Reference" "J8" (at 45.72 132.08 0)
+    (property "Reference" "J8" (at 45.72 134.62 0)
       (effects (font (size 1.27 1.27)))
     )
     (property "Value" "Conn_02x04_Counter_Clockwise" (at 45.72 134.62 0)
-      (effects (font (size 1.27 1.27)))
+      (effects (font (size 1.27 1.27)) hide)
     )
     (property "Footprint" "" (at 44.45 140.97 0)
