File: schematics/MC68000/uart_control.kicad_sch (KiCad schematic)
At the start: 4 parts, among them J11 Conn_02x20_Counter_Clockwise, J12 Conn_02x37_Row_Letter_Last, U28 74LS139, U29 74LS138

Commit message: Updating...
Connections:
- net key_cs: now reaches U29.11 (O4)
- net key_cs: now also J12.32b (Pin_32b)
Changed lines of the file:
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@@
+    (stroke (width 0) (type default))
+  )
+  (wire (pts (xy 168.91 120.65) (xy 163.83 120.65))
     (stroke (width 0) (type default))
   )
@@
     (effects (font (size 1.27 1.27)) (justify left bottom))
   )
+  (global_label "key_cs" (shape input) (at 55.88 50.8 0) (fields_autoplaced)
+    (effects (font (size 1.27 1.27)) (justify left))
+    (property "Intersheetrefs" "${INTERSHEET_REFS}" (at 65.0338 50.8 0)
+      (effects (font (size 1.27 1.27)) (justify left) hide)
+    )
+  )
   (global_label "bD1" (shape input) (at 60.96 90.17 0) (fields_autoplaced)
     (effects (font (size 1.27 1.27)) (justify left))
@@
     )
   )
+  (global_label "key_cs" (shape input) (at 168.91 120.65 0) (fields_autoplaced)
+    (effects (font (size 1.27 1.27)) (justify left))
+    (property "Intersheetrefs" "${INTERSHEET_REFS}" (at 178.0638 120.65 0)
+      (effects (font (size 1.27 1.27)) (justify left) hide)
+    )
+  )

Commit message: Update 2025/08/14
Other:
- note added: "UART1 - 0x4000 até 0x20FF = UART_CS1 UART2 - 0x4100 até 0x21FF = UART_CS2 UART3 - 0x4200 até 0x22FF = UART_CS3 UART4 - 0x4300 até 0x23FF = UART_CS4 key - 0x4400 até 0x44ff = key_cs na leitura Led - 0x4400 até 0x44ff = LED_CS na escrita"
- note removed: "UART1 - 0x2000 até 0x20FF = UART_CS1 UART2 - 0x2100 até 0x21FF = UART_CS2 UART3 - 0x2200 até 0x22FF = UART_CS3 UART4 - 0x2300 até 0x23FF = UART_CS4"
Changed lines of the file:
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@@
     (stroke (width 0) (type default))
   )
-  (text "UART1 - 0x2000 até 0x20FF = UART_CS1                  \nUART2 - 0x2100 até 0x21FF = UART_CS2                                                   \nUART3 - 0x2200 até 0x22FF = UART_CS3                                                   \nUART4 - 0x2300 até 0x23FF = UART_CS4\n"
-    (at 22.86 24.13 0)
+  (text "UART1 - 0x4000 até 0x20FF = UART_CS1                  \nUART2 - 0x4100 até 0x21FF = UART_CS2                                                   \nUART3 - 0x4200 até 0x22FF = UART_CS3                                                   \nUART4 - 0x4300 até 0x23FF = UART_CS4\nkey   - 0x4400 até 0x44ff = key_cs   na leitura\nLed   - 0x4400 até 0x44ff = LED_CS   na escrita"
+    (at 19.05 30.48 0)
     (effects (font (size 1.27 1.27)) (justify left bottom))
   )

Commit message: update...
Connections:
- net bE is gone; now on net /WRL: J12.19b (Pin_19b)
- net IRQ1: now also J12.5b (Pin_5b); no longer J12.6b (Pin_6b)
- net IRQ2: now also J12.6b (Pin_6b); no longer J12.7b (Pin_7b)
- net IRQ3: now also J12.7b (Pin_7b); no longer J12.8b (Pin_8b)
- net IRQ6: now also J12.8b (Pin_8b); no longer J12.11b (Pin_11b)
- net /RDL: now also J12.28b (Pin_28b)
- net IRQ4 renamed IACK1
- net IRQ5 renamed IACK2
- net IRQ7 renamed IACK6
- new net IACK3: J12.11b (Pin_11b)
Changed lines of the file:
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@@
-    (stroke (width 0) (type default))
-  )
-  (bus_entry (at 176.53 85.09) (size -2.54 2.54)
     (stroke (width 0) (type default))
   )
@@
     (stroke (width 0) (type default))
   )
-  (bus (pts (xy 176.53 83.82) (xy 176.53 85.09))
+  (bus (pts (xy 176.53 83.82) (xy 176.53 87.63))
     (stroke (width 0) (type default))
   )
@@
     (stroke (width 0) (type default))
   )
+  (wire (pts (xy 180.34 110.49) (xy 181.61 110.49))
+    (stroke (width 0) (type default))
+  )
   (wire (pts (xy 60.96 105.41) (xy 52.07 105.41))
     (stroke (width 0) (type default))
@@
     (stroke (width 0) (type default))
   )
-  (wire (pts (xy 173.99 87.63) (xy 163.83 87.63))
-    (stroke (width 0) (type default))
-  )
   (wire (pts (xy 60.96 102.87) (xy 52.07 102.87))
     (stroke (width 0) (type default))
@@
     (stroke (width 0) (type default))
   )
-  (bus (pts (xy 176.53 85.09) (xy 176.53 87.63))
-    (stroke (width 0) (type default))
-  )
   (wire (pts (xy 135.89 95.25) (xy 151.13 95.25))
     (stroke (width 0) (type default))
@@
     (stroke (width 0) (type default))
   )
+  (wire (pts (xy 163.83 110.49) (xy 180.34 110.49))
+    (stroke (width 0) (type default))
+  )
   (wire (pts (xy 173.99 92.71) (xy 163.83 92.71))
     (stroke (width 0) (type default))
@@
     (stroke (width 0) (type default))
   )
+  (wire (pts (xy 176.53 87.63) (xy 163.83 87.63))
+    (stroke (width 0) (type default))
+  )
   (wire (pts (xy 139.7 49.53) (xy 151.13 49.53))
     (stroke (width 0) (type default))
@@
   )
   (bus (pts (xy 133.35 95.25) (xy 133.35 97.79))
+    (stroke (width 0) (type default))
+  )
+  (wire (pts (xy 181.61 87.63) (xy 176.53 87.63))
     (stroke (width 0) (type default))
   )
@@
     (effects (font (size 1.27 1.27)) (justify left bottom))
   )
-  (label "IRQ3" (at 163.83 59.69 0) (fields_autoplaced)
+  (label "IACK3" (at 163.83 67.31 0) (fields_autoplaced)
+    (effects (font (size 1.27 1.27)) (justify left bottom))
+  )
+  (label "IRQ3" (at 163.83 57.15 0) (fields_autoplaced)
     (effects (font (size 1.27 1.27)) (justify left bottom))
   )
@@
     (effects (font (size 1.27 1.27)) (justify left bottom))
   )
-  (label "IRQ6" (at 163.83 67.31 0) (fields_autoplaced)
+  (label "IRQ6" (at 163.83 59.69 0) (fields_autoplaced)
     (effects (font (size 1.27 1.27)) (justify left bottom))
   )
@@
     (effects (font (size 1.27 1.27)) (justify left bottom))
   )
-  (label "IRQ1" (at 163.83 54.61 0) (fields_autoplaced)
+  (label "IRQ1" (at 163.83 52.07 0) (fields_autoplaced)
     (effects (font (size 1.27 1.27)) (justify left bottom))
   )
@@
   )
   (label "bD13" (at 139.7 128.27 0) (fields_autoplaced)
-    (effects (font (size 1.27 1.27)) (justify left bottom))
-  )
-  (label "bE" (at 163.83 87.63 0) (fields_autoplaced)
     (effects (font (size 1.27 1.27)) (justify left bottom))
   )
@@
     (effects (font (size 1.27 1.27)) (justify left bottom))
   )
-  (label "IRQ2" (at 163.83 57.15 0) (fields_autoplaced)
+  (label "IRQ2" (at 163.83 54.61 0) (fields_autoplaced)
     (effects (font (size 1.27 1.27)) (justify left bottom))
   )
@@
     (effects (font (size 1.27 1.27)) (justify left bottom))
   )
-  (label "IRQ7" (at 163.83 69.85 0) (fields_autoplaced)
-    (effects (font (size 1.27 1.27)) (justify left bottom))
-  )
   (label "bD15" (at 139.7 133.35 0) (fields_autoplaced)
     (effects (font (size 1.27 1.27)) (justify left bottom))
@@
   )
   (label "bD6" (at 139.7 110.49 0) (fields_autoplaced)
+    (effects (font (size 1.27 1.27)) (justify left bottom))
+  )
+  (label "IACK6" (at 163.83 69.85 0) (fields_autoplaced)
     (effects (font (size 1.27 1.27)) (justify left bottom))
   )
@@
     (effects (font (size 1.27 1.27)) (justify left bottom))
   )
-  (label "IRQ4" (at 163.83 62.23 0) (fields_autoplaced)
-    (effects (font (size 1.27 1.27)) (justify left bottom))
-  )
   (label "{slash}WR" (at 163.83 100.33 0) (fields_autoplaced)
     (effects (font (size 1.27 1.27)) (justify left bottom))
@@
     (effects (font (size 1.27 1.27)) (justify right bottom))
   )
+  (label "IACK1" (at 163.83 62.23 0) (fields_autoplaced)
+    (effects (font (size 1.27 1.27)) (justify left bottom))
+  )
+  (label "IACK2" (at 163.83 64.77 0) (fields_autoplaced)
+    (effects (font (size 1.27 1.27)) (justify left bottom))
+  )
   (label "bA6" (at 139.7 54.61 0) (fields_autoplaced)
     (effects (font (size 1.27 1.27)) (justify left bottom))
@@
   )
   (label "bD9" (at 139.7 118.11 0) (fields_autoplaced)
-    (effects (font (size 1.27 1.27)) (justify left bottom))
-  )
-  (label "IRQ5" (at 163.83 64.77 0) (fields_autoplaced)
     (effects (font (size 1.27 1.27)) (justify left bottom))
   )
@@
     )
   )
+  (global_label "{slash}WRL" (shape input) (at 181.61 87.63 0) (fields_autoplaced)
+    (effects (font (size 1.27 1.27)) (justify left))
+    (property "Intersheetrefs" "${INTERSHEET_REFS}" (at 189.6752 87.63 0)
+      (effects (font (size 1.27 1.27)) (justify left) hide)
+    )
+  )
   (global_label "{slash}UART_CS1" (shape input) (at 60.96 118.11 0) (fields_autoplaced)
     (effects (font (size 1.27 1.27)) (justify left))
@@
       (effects (font (size 1.27 1.27)) (justify left) hide)
     )
+  )
+  (global_label "{slash}RDL" (shape input) (at 181.61 110.49 0) (fields_autoplaced)
+    (effects (font (size 1.27 1.27)) (justify left))
+    (property "Intersheetrefs" "${INTERSHEET_REFS}" (at 189.4938 110.49 0)
+      (effects (font (size 1.27 1.27)) (justify left) hide)
+    )

Commit message: updating
Connections:
- net /bLDS: no longer U28.1 (E)
- net /bUDS: now also U28.1 (E)
Changed lines of the file:
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@@
 		)
 	)
-	(label "{slash}bLDS"
+	(label "{slash}bUDS"
 		(at 111.76 105.41 0)
 		(effects
